File: life-cell/Cell.kicad_sch (KiCad schematic)
At the start: 7 parts, among them J5 UPDI, SW1 Toggle, U1 ATtiny404-SS

Commit message: Fix LED resistor value
Parts:
- R1: value 1k -> 120R
Changed lines of the file:
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@@
     (in_bom yes) (on_board yes) (fields_autoplaced)
     (property "Reference" "R1" (id 0) (at 180.34 71.12 90))
-    (property "Value" "1k" (id 1) (at 180.34 73.66 90))
+    (property "Value" "120R" (id 1) (at 180.34 73.66 90))
     (property "Footprint" "Resistor_SMD:R_0603_1608Metric_Pad0.98x0.95mm_HandSolder" (id 2) (at 180.34 79.248 90)
       (effects (font (size 1.27 1.27)) hide)
