File: life-cell/life-cell.kicad_pcb (KiCad board)
At the start: 2 copper layers, 44.4 x 44.4 mm, 15 parts, among them J1 Interconnect, J2 Interconnect, J3 Interconnect, J4 Interconnect, J5 UPDI, SW1 Toggle, U1 ATtiny404-SS

Commit message: Fix LED resistor value
Parts:
- R1: value 1k -> 120R
Changed lines of the file:
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@@
       (effects (font (size 1 1) (thickness 0.15)))
     )
-    (fp_text value "1k" (at 0 1.43 90) (layer "F.Fab")
+    (fp_text value "120R" (at 0 1.43 90) (layer "F.Fab")
       (effects (font (size 1 1) (thickness 0.15)))
     )
