File: life-cell/pcb/life-cell.kicad_pcb (KiCad board)
At the start: 2 copper layers, 44.4 x 44.4 mm, 15 parts, among them J1 Interconnect, J2 Interconnect, J3 Interconnect, J4 Interconnect, J5 UPDI, SW1 Toggle, U1 ATtiny404-SS

Commit message: Add NSEW schem/silkscreen labels
Other:
- board text added: "EAST"
- board text added: "NORTH"
- board text added: "SOUTH"
- board text added: "WEST"
Changed lines of the file:
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@@
     (property "P/N" "")
     (property "Sheetfile" "Interconnect.kicad_sch")
-    (property "Sheetname" "Interconnect3")
+    (property "Sheetname" "Interconnect3-South")
     (attr through_hole)
     (fp_text reference "J3" (at 0 2.33 270 unlocked) (layer "B.SilkS")
@@
     (property "P/N" "")
     (property "Sheetfile" "Interconnect.kicad_sch")
-    (property "Sheetname" "Interconnect4")
+    (property "Sheetname" "Interconnect4-West")
     (attr through_hole)
     (fp_text reference "J4" (at 0 2.33 180 unlocked) (layer "B.SilkS")
@@
     (property "P/N" "")
     (property "Sheetfile" "Interconnect.kicad_sch")
-    (property "Sheetname" "Interconnect1")
+    (property "Sheetname" "Interconnect1-North")
     (attr through_hole)
     (fp_text reference "J1" (at 0 2.33 90 unlocked) (layer "B.SilkS")
@@
     (property "P/N" "")
     (property "Sheetfile" "Interconnect.kicad_sch")
-    (property "Sheetname" "Interconnect2")
+    (property "Sheetname" "Interconnect2-East")
     (attr through_hole)
     (fp_text reference "J2" (at 0 2.33 unlocked) (layer "B.SilkS")
@@
   (gr_line (start 170.815 83.185) (end 170.815 41.275) (layer "Edge.Cuts") (width 0.1))
   (gr_arc (start 215.265 83.185) (mid 214.893026 84.083026) (end 213.995 84.455) (layer "Edge.Cuts") (width 0.1))
-  (gr_text "Adam Gausmann" (at 206.248 52.578) (layer "B.SilkS")
+  (gr_text "Adam Gausmann" (at 205.74 53.848) (layer "B.SilkS")
     (effects (font (size 1 1) (thickness 0.15)) (justify left mirror))
   )
@@
     (effects (font (size 1 1) (thickness 0.15)) (justify right mirror))
   )
-  (gr_text "Life Cell" (at 196.088 51.054) (layer "B.SilkS")
+  (gr_text "NORTH" (at 193.04 49.403) (layer "B.SilkS")
+    (effects (font (size 1 1) (thickness 0.15)) (justify mirror))
+  )
+  (gr_text "SOUTH" (at 193.04 75.057 180) (layer "B.SilkS")
+    (effects (font (size 1 1) (thickness 0.15)) (justify mirror))
+  )
+  (gr_text "Life Cell" (at 195.58 52.324) (layer "B.SilkS")
     (effects (font (size 1 1) (thickness 0.15)) (justify left mirror))
   )
-  (gr_text "HWLife" (at 206.502 50.546) (layer "B.SilkS")
+  (gr_text "HWLife" (at 205.994 51.816) (layer "B.SilkS")
     (effects (font (size 2 2) (thickness 0.3)) (justify left mirror))
   )
@@
     (effects (font (size 1 1) (thickness 0.15)) (justify right mirror))
   )
+  (gr_text "WEST" (at 180.213 62.23 90) (layer "B.SilkS")
+    (effects (font (size 1 1) (thickness 0.15)) (justify mirror))
+  )
   (gr_text "GND\n" (at 199.898 73.66) (layer "B.SilkS")
     (effects (font (size 1 1) (thickness 0.15)) (justify right mirror))
   )
-  (gr_text "2022-10-22" (at 206.248 54.102) (layer "B.SilkS")
+  (gr_text "EAST" (at 205.867 62.23 270) (layer "B.SilkS")
+    (effects (font (size 1 1) (thickness 0.15)) (justify mirror))
+  )
+  (gr_text "2022-10-22" (at 205.74 55.372) (layer "B.SilkS")
     (effects (font (size 1 1) (thickness 0.15)) (justify left mirror))
   )
