File: life-cell/pcb/life-cell.kicad_pcb (KiCad board)
At the start: 2 copper layers, 44.4 x 44.4 mm, 15 parts, among them J1 Interconnect, J2 Interconnect, J3 Interconnect, J4 Interconnect, J5 UPDI, SW1 Toggle, U1 ATtiny404-SS

Commit message: Switch to "symmetric" connector layout.
Each side has half male pins and half female pins, for a truly
symmetric experience!
Parts:
- added J6: Interconnect In, Connector_PinHeader_2.54mm:PinHeader_1x05_P2.54mm_Horizontal, B.Cu at (194.3, 77.5)
- added J7: Interconnect Out, Connector_PinSocket_2.54mm:PinSocket_1x05_P2.54mm_Horizontal, B.Cu at (191.8, 77.5)
- added J8: Interconnect In, Connector_PinHeader_2.54mm:PinHeader_1x05_P2.54mm_Horizontal, B.Cu at (208.3, 61.0)
- added J9: Interconnect Out, Connector_PinSocket_2.54mm:PinSocket_1x05_P2.54mm_Horizontal, B.Cu at (208.3, 63.5)
- J1: value Interconnect -> UPDI; footprint Connector_PinHeader_2.54mm:PinHeader_1x10_P2.54mm_Vertical -> Connector_PinHeader_2.54mm:PinHeader_1x03_P2.54mm_Vertical
- J2, J4: value Interconnect -> Interconnect In; footprint Connector_PinHeader_2.54mm:PinHeader_1x10_P2.54mm_Vertical -> Connector_PinHeader_2.54mm:PinHeader_1x05_P2.54mm_Horizontal
- J3: value Interconnect -> Interconnect Out; footprint Connector_PinHeader_2.54mm:PinHeader_1x10_P2.54mm_Vertical -> Connector_PinSocket_2.54mm:PinSocket_1x05_P2.54mm_Horizontal
- J5: value UPDI -> Interconnect Out; footprint Connector_PinHeader_2.54mm:PinHeader_1x03_P2.54mm_Vertical -> Connector_PinSocket_2.54mm:PinSocket_1x05_P2.54mm_Horizontal
- moved J3 32.1 mm to (194.3, 47.0), turned to -90 degrees
- moved J1 27.2 mm to (198.1, 68.6), turned to 180 degrees
- moved J5 21.7 mm to (177.8, 61.0), turned to 0 degrees
- moved J2 16.9 mm to (191.8, 47.0), turned to 90 degrees
- moved J4 10.2 mm to (177.8, 63.5), turned to 180 degrees
Connections:
- J1 pad 1: /Cell/DIA1 -> VCC
- J1 pad 2: /Cell/ADJ1 -> /Cell/NRST
- J2 pad 1: /Cell/DIA2 -> VCC
- J2 pad 2: /Cell/ADJ2 -> /Cell/CLK
- J2 pad 4: /Cell/CLK -> /Cell/ADJ1
- J2 pad 5: VCC -> /Cell/DIA1
- J3 pad 1: /Cell/DIA3 -> VCC
- J3 pad 2: /Cell/ADJ3 -> /Cell/CLK
- J3 pad 4: /Cell/CLK -> /Cell/STATE
- J3 pad 5: VCC -> /Cell/ADJ2
- J4 pad 1: /Cell/DIA4 -> VCC
- J4 pad 2: /Cell/ADJ4 -> /Cell/CLK
- J4 pad 4: /Cell/CLK -> /Cell/ADJ4
- J4 pad 5: VCC -> /Cell/DIA4
- J5 pad 2: /Cell/NRST -> /Cell/CLK
