File: modular-backplane/backplane/Cell.kicad_sch (KiCad schematic)
At the start: 1 part, among them J9 Module

Commit message: Place and route power/management connectors and power switch
Connections:
- net NRST: now reaches J9.9 (Pin_9)
- no-connect marks 1 -> 0
Changed lines of the file:
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@@
   (junction (at 95.25 48.26) (diameter 0) (color 0 0 0 0)
   )
-  (no_connect (at 59.69 73.66))
   (wire (pts (xy 95.25 58.42) (xy 95.25 55.88))
     (stroke (width 0) (type default) (color 0 0 0 0))
@@
     (effects (font (size 1.27 1.27)) (justify left bottom))
   )
+  (global_label "NRST" (shape input) (at 59.69 73.66 180) (fields_autoplaced)
+    (effects (font (size 1.27 1.27)) (justify right))
+    (property "Intersheet References" "${INTERSHEET_REFS}" (id 0) (at 52.4993 73.5806 0)
+      (effects (font (size 1.27 1.27)) (justify right) hide)
+    )
+  )
   (global_label "VLED" (shape input) (at 54.61 81.28 180) (fields_autoplaced)

Commit message: Place and route clock tree; remove NRST from management header
Changed lines of the file:
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@@
+    (stroke (width 0) (type default) (color 0 0 0 0))
+  )
+  (wire (pts (xy 48.26 73.66) (xy 59.69 73.66))
     (stroke (width 0) (type default) (color 0 0 0 0))
   )
@@
     (effects (font (size 1.27 1.27)) (justify right bottom))
   )
+  (label "NRST" (at 48.26 73.66 0)
+    (effects (font (size 1.27 1.27)) (justify left bottom))
+  )
   (label "STATE" (at 88.9 38.1 0)
     (effects (font (size 1.27 1.27)) (justify left bottom))
   )
-  (global_label "NRST" (shape input) (at 59.69 73.66 180) (fields_autoplaced)
-    (effects (font (size 1.27 1.27)) (justify right))
-    (property "Intersheet References" "${INTERSHEET_REFS}" (id 0) (at 52.4993 73.5806 0)
-      (effects (font (size 1.27 1.27)) (justify right) hide)
-    )
-  )
   (global_label "VLED" (shape input) (at 54.61 81.28 180) (fields_autoplaced)
