File: modular-backplane/backplane/backplane.kicad_pcb (KiCad board)
At the start: 4 copper layers, 100 x 100 mm, 86 parts, among them J1 West, J10 Module, J11 Module, J12 Module, J13 Module, J14 Module, J15 Module, J16 Module, J17 Module, J18 Module, J19 Module, J2 South, J20 Module, J21 Module, J22 Module, J23 Module, J24 Module, J25 Module, J26 Module, J27 Module, J28 Module, J29 Module, J3 North, J30 Module, J31 Module, J32 Module, J33 Module, J34 Module, J35 Module, J36 Module, J37 Module, J38 Module, J39 Module, J4 East, J40 Module, J41 Module, J42 Module, J43 Module, J44 Module, J45 Module, J46 Module, J47 Module, J48 Module, J49 Module, J5 25-E900-02, J50 Module, J51 Module, J52 Module, J53 Module, J54 Module, J55 Module, J56 Module, J57 Module, J58 Module, J59 Module, J6 MGMT, J60 Module, J61 Module, J62 Module, J63 Module, J64 Module, J65 Module, J66 Module, J67 Module, J68 Module, J69 Module, J70 Module, J71 Module, J72 Module, J9 Module, SW1 A, SW2 B, SW3 C, SW4 D, SW5 E, SW6 F, SW7 G, SW8 H, U1 74HC14, U2 74HC14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

Commit message: Backplane finishing touches
Other:
- board text added: "+5V"
- board text added: "Adam Gausmann"
- board text added: "East"
- board text added: "GND"
- board text added: "GND +5V CLK DIM"
- board text added: "HWLife Backplane"
- board text added: "North"
- board text added: "Rev1 2023-01-23"
- board text added: "South"
- board text added: "West"

Commit message: Add PTC fuse; add orientation marks for modules
Parts:
- added F1: 6V 3A, Fuse:Fuse_1812_4532Metric_Pad1.30x3.40mm_HandSolder, B.Cu at (77.9, 80.9)
Connections:
- J5 pad 2: +5V -> /5V_IN
Routing:
- net /CLK1: track 108.4 -> 83.7 mm
- net /T-C1: track 23.4 -> 32.8 mm
- net /T-C0: track 35.6 -> 44.7 mm
- net /5V_IN: track 0.00 -> 6.63 mm
- net +5V: track 1636.5 -> 1638.3 mm, vias 66 -> 65
Other:
- board text added: "Rev1 2023-02-07"
- board text removed: "Rev1 2023-01-23"
