File: modular-backplane/backplane/backplane.kicad_sch (KiCad schematic)
At the start: 22 parts, among them J1 West, J2 South, J3 North, J4 East, J5 25-E900-02, J6 MGMT, SW1 A, SW2 B, SW3 C, SW4 D, SW5 E, SW6 F, SW7 G, SW8 H, U1 74HC14, U2 74HC14, U3 VN5E160S

Commit message: Add PTC fuse; add orientation marks for modules
Parts:
- added F1: 6V 3A, Fuse:Fuse_1812_4532Metric_Pad1.30x3.40mm_HandSolder, symbol Device:Polyfuse
Connections:
- net +5V: now also F1.2; no longer J5.2 (Pin_2)
- new net 5V_IN: F1.1, J5.2 (Pin_2)
Changed lines of the file:
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@@
   (junction (at 472.44 306.07) (diameter 0) (color 0 0 0 0)
   )
+  (junction (at 463.55 177.8) (diameter 0) (color 0 0 0 0)
+  )
   (junction (at 345.44 284.48) (diameter 0) (color 0 0 0 0)
   )
@@
     (stroke (width 0) (type default) (color 0 0 0 0))
   )
+  (wire (pts (xy 463.55 177.8) (xy 471.17 177.8))
+    (stroke (width 0) (type default) (color 0 0 0 0))
+  )
   (wire (pts (xy 200.66 144.78) (xy 200.66 149.86))
     (stroke (width 0) (type default) (color 0 0 0 0))
@@
     (stroke (width 0) (type default) (color 0 0 0 0))
   )
+  (wire (pts (xy 478.79 177.8) (xy 485.14 177.8))
+    (stroke (width 0) (type default) (color 0 0 0 0))
+  )
   (wire (pts (xy 322.58 144.78) (xy 322.58 149.86))
     (stroke (width 0) (type default) (color 0 0 0 0))
@@
     (stroke (width 0) (type default) (color 0 0 0 0))
   )
+  (wire (pts (xy 461.01 177.8) (xy 463.55 177.8))
+    (stroke (width 0) (type default) (color 0 0 0 0))
+  )
   (wire (pts (xy 213.36 274.32) (xy 213.36 269.24))
     (stroke (width 0) (type default) (color 0 0 0 0))
@@
     (stroke (width 0) (type default) (color 0 0 0 0))
   )
+  (wire (pts (xy 463.55 177.8) (xy 463.55 180.34))
+    (stroke (width 0) (type default) (color 0 0 0 0))
+  )
   (wire (pts (xy 139.7 175.26) (xy 139.7 180.34))
     (stroke (width 0) (type default) (color 0 0 0 0))
@@
     (effects (font (size 1.27 1.27)) (justify right bottom))
   )
+  (label "5V_IN" (at 463.55 180.34 0)
+    (effects (font (size 1.27 1.27)) (justify left bottom))
+  )
   (label "T-C5" (at 285.75 160.02 180)
     (effects (font (size 1.27 1.27)) (justify right bottom))
@@
     (pin "9")
   )
-  (symbol (lib_id "power:+5V") (at 461.01 177.8 270) (unit 1)
+  (symbol (lib_id "power:+5V") (at 485.14 177.8 270) (unit 1)
     (in_bom yes) (on_board yes) (fields_autoplaced)
-    (property "Reference" "#PWR0109" (id 0) (at 457.2 177.8 0)
+    (property "Reference" "#PWR0109" (id 0) (at 481.33 177.8 0)
       (effects (font (size 1.27 1.27)) hide)
     )
-    (property "Value" "+5V" (id 1) (at 464.82 177.7999 90)
+    (property "Value" "+5V" (id 1) (at 488.95 177.7999 90)
       (effects (font (size 1.27 1.27)) (justify left))
     )
-    (property "Footprint" "" (id 2) (at 461.01 177.8 0)
+    (property "Footprint" "" (id 2) (at 485.14 177.8 0)
       (effects (font (size 1.27 1.27)) hide)
     )
-    (property "Datasheet" "" (id 3) (at 461.01 177.8 0)
+    (property "Datasheet" "" (id 3) (at 485.14 177.8 0)
       (effects (font (size 1.27 1.27)) hide)
     )
@@
     (pin "1")
   )
+  (symbol (lib_id "Device:Polyfuse") (at 474.98 177.8 90) (unit 1)
+    (in_bom yes) (on_board yes) (fields_autoplaced)
+    (property "Reference" "F1" (id 0) (at 474.98 171.45 90))
+    (property "Value" "6V 3A" (id 1) (at 474.98 173.99 90))
+    (property "Footprint" "Fuse:Fuse_1812_4532Metric_Pad1.30x3.40mm_HandSolder" (id 2) (at 480.06 176.53 0)
+      (effects (font (size 1.27 1.27)) (justify left) hide)
+    )
+    (property "Datasheet" "~" (id 3) (at 474.98 177.8 0)
+      (effects (font (size 1.27 1.27)) hide)
+    )
+    (property "Digikey" "283-3166-1-ND" (id 4) (at 474.98 177.8 0)
+      (effects (font (size 1.27 1.27)) hide)
+    )
+    (property "Manufacturer" "Eaton" (id 5) (at 474.98 177.8 0)
+      (effects (font (size 1.27 1.27)) hide)
+    )
+    (property "Mfr. Part #" "PTS18126V300" (id 6) (at 474.98 177.8 0)
+      (effects (font (size 1.27 1.27)) hide)
+    )
+    (pin "1")
+    (pin "2")
+  )
   (symbol (lib_id "power:+5V") (at 528.32 138.43 0) (unit 1)
     (in_bom yes) (on_board yes) (fields_autoplaced)
@@
       (reference "#PWR0213") (unit 1) (value "GND") (footprint "")
     )
+    (path "/48cd7377-dc26-4d50-b2ad-989ab2474676"
+      (reference "F1") (unit 1) (value "6V 3A") (footprint "Fuse:Fuse_1812_4532Metric_Pad1.30x3.40mm_HandSolder")
+    )
     (path "/852e5412-4b34-47d4-9b60-8d540a352e29"
