File: modular-backplane/single-cell/single-cell.kicad_sch (KiCad schematic)
At the start: 6 parts, among them J1 To Backplane, U1 ATtiny404-SS

Commit message: Update some component details
Parts:
- removed J1: To Backplane, agausmann:Molex_SlimStack_216701-0209_02x10_P0.35mm_Vertical, symbol Connector_Generic:Conn_02x10_Odd_Even
- added J?: To Backplane, symbol Connector_Generic:Conn_02x08_Odd_Even

Commit message: (Re)route single-cell module; add grabbing holes and markings
Parts:
- added H1, H2: Pull, agausmann:Hole_Cell, symbol Mechanical:MountingHole
- J1: renamed from J?; footprint (none) -> agausmann:XKB_X1321FVS_02x08_P1.27mm_Vertical
Connections:
- net TOGGLE is gone; now on net CLK: U1.2 (PA4)
- net VCC is gone; now on net +5V: C1.1, C2.1, U1.1 (VCC)
- net CLK: now also J1.11 (Pin_11)
- net GND: now also J1.14 (Pin_14), J1.16 (Pin_16)
- net NRST: now also J1.9 (Pin_9)
- net STATE: now also J1.10 (Pin_10)
- net VLED: now also J1.15 (Pin_15)
- net IN7: now reaches J1.1 (Pin_1)
- net IN7: now also U1.7 (PB2)
- net INIT: now reaches J1.12 (Pin_12)
- net INIT: now also U1.13 (PA3)
- net +5V: now reaches J1.13 (Pin_13)
- net IN6: now reaches J1.2 (Pin_2)
- net IN6: now also U1.8 (PB1)
- net IN0: now reaches J1.3 (Pin_3)
- net IN0: now also U1.6 (PB3)
- net IN5: now reaches J1.4 (Pin_4)
- net IN5: now also U1.9 (PB0)
- net IN1: now reaches J1.5 (Pin_5)
- net IN1: now also U1.5 (PA7)
- net IN4: now reaches J1.6 (Pin_6)
- net IN4: now also U1.11 (PA1)
- net IN2: now reaches J1.7 (Pin_7)
- net IN2: now also U1.4 (PA6)
- net IN3: now reaches J1.8 (Pin_8)
- net IN3: now also U1.12 (PA2)
